File: MCU_DataLogger.kicad_sch (KiCad schematic)
At the start: 25 parts, among them U1 24LC1025, U2 24LC1025, U3 ATMEGA328P-AU, U4 DS1337S_, Y1 32.768 KHz, Y2 16 MHz

Commit message: 2-layer PCB complete
Connections:
- net Vcc is gone; now on net VCC: C1.1, R1.1, R2.1, R3.1, R6.1, R7.1, U1.1 (A0), U1.2 (A1), U1.3 (A2), U1.8 (VCC), U2.1 (A0), U2.3 (A2), U2.8 (VCC), U4.8 (VCC)
- net SCK: no longer R6.2, U1.6 (SCL), U2.6 (SCL), U3.28 (PC5), U4.6 (SCL)
- new net SCL: R6.2, U1.6 (SCL), U2.6 (SCL), U3.28 (PC5), U4.6 (SCL)
Other:
- sheet connectors ports: added SCL; removed none
Changed lines of the file:
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@@
 	)
 	(junction
-		(at 255.27 40.64)
+		(at 240.03 40.64)
 		(diameter 0)
 		(color 0 0 0 0)
@@
 	(wire
 		(pts
-			(xy 251.46 40.64) (xy 233.68 40.64)
+			(xy 233.68 40.64) (xy 240.03 40.64)
 		)
 		(stroke
@@
 	(wire
 		(pts
+			(xy 240.03 36.83) (xy 240.03 40.64)
+		)
+		(stroke
+			(width 0)
+			(type default)
+		)
+	)
+	(wire
+		(pts
 			(xy 100.33 140.97) (xy 105.41 140.97)
 		)
@@
 	(wire
 		(pts
-			(xy 134.62 143.51) (xy 140.97 143.51)
+			(xy 134.62 144.78) (xy 140.97 144.78)
 		)
 		(stroke
@@
 	(wire
 		(pts
+			(xy 134.62 138.43) (xy 140.97 138.43)
+		)
+		(stroke
+			(width 0)
+			(type default)
+		)
+	)
+	(wire
+		(pts
 			(xy 81.28 162.56) (xy 81.28 165.1)
 		)
@@
 	(wire
 		(pts
-			(xy 134.62 140.97) (xy 140.97 140.97)
+			(xy 134.62 142.24) (xy 140.97 142.24)
 		)
 		(stroke
@@
 	(wire
 		(pts
+			(xy 240.03 40.64) (xy 251.46 40.64)
+		)
+		(stroke
+			(width 0)
+			(type default)
+		)
+	)
+	(wire
+		(pts
 			(xy 271.78 44.45) (xy 271.78 40.64)
 		)
@@
 	(wire
 		(pts
-			(xy 259.08 40.64) (xy 255.27 40.64)
+			(xy 251.46 40.64) (xy 259.08 40.64)
 		)
 		(stroke
@@
 	(wire
 		(pts
-			(xy 255.27 40.64) (xy 251.46 40.64)
-		)
-		(stroke
-			(width 0)
-			(type default)
-		)
-	)
-	(wire
-		(pts
 			(xy 119.38 46.99) (xy 125.73 46.99)
 		)
@@
 		)
 	)
-	(label "Vcc"
-		(at 71.12 152.4 180)
-		(effects
-			(font
-				(size 1.27 1.27)
-			)
-			(justify right bottom)
-		)
-	)
 	(label "TX"
-		(at 134.62 140.97 180)
+		(at 134.62 142.24 180)
 		(effects
 			(font
@@
 		)
 	)
-	(label "Vcc"
-		(at 38.1 154.94 180)
-		(effects
-			(font
-				(size 1.27 1.27)
-			)
-			(justify right bottom)
-		)
-	)
 	(label "SCK"
 		(at 203.2 68.58 180)
@@
 		)
 	)
-	(label "SCK"
+	(label "SCL"
 		(at 58.42 154.94 0)
 		(effects
@@
 		)
 	)
-	(label "SCK"
+	(label "SCL"
 		(at 100.33 161.29 0)
 		(effects
@@
 		)
 	)
-	(label "SCK"
+	(label "Vcc"
+		(at 38.1 154.94 180)
+		(effects
+			(font
+				(size 1.27 1.27)
+			)
+			(justify right bottom)
+		)
+	)
+	(label "SCL"
 		(at 134.62 134.62 180)
 		(effects
@@
 	)
 	(label "RX"
-		(at 134.62 143.51 180)
+		(at 134.62 144.78 180)
 		(effects
 			(font
@@
 		)
 	)
-	(label "SCK"
+	(label "SCL"
 		(at 91.44 154.94 0)
 		(effects
@@
 		)
 	)
+	(label "SCK"
+		(at 134.62 138.43 180)
+		(effects
+			(font
+				(size 1.27 1.27)
+			)
+			(justify right bottom)
+		)
+	)
 	(label "Vcc"
 		(at 105.41 134.62 0)
@@
 		)
 	)
-	(label "SCK"
+	(label "SCL"
 		(at 74.93 52.07 180)
 		(effects
@@
 		)
 	)
+	(label "Vcc"
+		(at 240.03 36.83 0)
+		(effects
+			(font
+				(size 1.27 1.27)
+			)
+			(justify left bottom)
+		)
+	)
 	(label "SDA"
 		(at 74.93 59.69 180)
@@
 		)
 	)
+	(label "Vcc"
+		(at 71.12 152.4 180)
+		(effects
+			(font
+				(size 1.27 1.27)
+			)
+			(justify right bottom)
+		)
+	)
 	(label "D5"
 		(at 176.53 135.89 0)
@@
 		)
 	)
-	(label "SCK"
+	(label "SCL"
 		(at 203.2 91.44 180)
 		(effects
@@
 	)
 	(symbol
-		(lib_id "power:PWR_FLAG")
-		(at 255.27 40.64 0)
-		(unit 1)
-		(body_style 1)
-		(exclude_from_sim no)
-		(in_bom yes)
-		(on_board yes)
-		(in_pos_files yes)
-		(dnp no)
-		(fields_autoplaced yes)
-		(property "Reference" "#FLG01"
-			(at 255.27 38.735 0)
-			(hide yes)
-			(show_name no)
-			(do_not_autoplace no)
-			(effects
-				(font
-					(size 1.27 1.27)
-				)
-			)
-		)
-		(property "Value" "PWR_FLAG"
-			(at 255.27 35.56 0)
-			(show_name no)
-			(do_not_autoplace no)
-			(effects
-				(font
-					(size 1.27 1.27)
-				)
-			)
-		)
-		(property "Footprint" ""
-			(at 255.27 40.64 0)
-			(hide yes)
-			(show_name no)
-			(do_not_autoplace no)
-			(effects
-				(font
-					(size 1.27 1.27)
-				)
-			)
-		)
-		(property "Datasheet" ""
-			(at 255.27 40.64 0)
-			(hide yes)
-			(show_name no)
-			(do_not_autoplace no)
-			(effects
-				(font
-					(size 1.27 1.27)
-				)
-			)
-		)
-		(property "Description" "Special symbol for telling ERC where power comes from"
-			(at 255.27 40.64 0)
-			(hide yes)
-			(show_name no)
-			(do_not_autoplace no)
-			(effects
-				(font
-					(size 1.27 1.27)
-				)
-			)
-		)
-		(pin "1"
-		)
-		(instances
-			(project "MCU_DataLogger"
-				(path "/eeff451f-3904-4ad2-8c5d-32d1f67f4fde"
-					(reference "#FLG01")
-					(unit 1)
-				)
-			)
-		)
-	)
-	(symbol
 		(lib_id "DS1337S_:DS1337S_")
 		(at 92.71 59.69 0)
@@
 		)
 		(pin "RX" input
-			(at 140.97 143.51 180)
+			(at 140.97 144.78 180)
 			(effects
 				(font
@@
 			)
 		)
-		(pin "SCK" passive
-			(at 140.97 134.62 180)
+		(pin "SDA" bidirectional
+			(at 140.97 132.08 180)
 			(effects
 				(font
@@
 			)
 		)
-		(pin "SDA" bidirectional
-			(at 140.97 132.08 180)
+		(pin "TX" output
+			(at 140.97 142.24 180)
 			(effects
 				(font
@@
 			)
 		)
-		(pin "TX" output
-			(at 140.97 140.97 180)
+		(pin "Vcc" passive
+			(at 140.97 127 180)
 			(effects
 				(font
@@
 			)
 		)
-		(pin "Vcc" passive
-			(at 140.97 127 180)
+		(pin "SCK" passive
+			(at 140.97 138.43 180)
+			(effects
+				(font
+					(size 1.27 1.27)
+				)
+				(justify left)
+			)
+		)
+		(pin "SCL" passive
+			(at 140.97 134.62 180)
 			(effects
 				(font
