File: MCU_DataLogger.kicad_sch (KiCad schematic)
At the start: 0 parts

Commit message: Schematic: add connectors sheet and custom library
Parts:
- added BT1: Battery, Connector_PinHeader_2.54mm:PinHeader_1x02_P2.54mm_Vertical, symbol Device:Battery
- added C1, C4: 0.1uF, Capacitor_SMD:C_0805_2012Metric, symbol Device:C
- added C2, C3: 22pF, Capacitor_SMD:C_0805_2012Metric, symbol Device:C
- added C5: 100nF, Capacitor_SMD:C_0805_2012Metric, symbol Device:C_Polarized
- added D1, D2: LED, LED_SMD:LED_0805_2012Metric, symbol Device:LED
- added H1, H2, H3, H4: MountingHole, MountingHole:MountingHole_2.1mm, symbol Mechanical:MountingHole
- added R1, R2, R3: 10K, Resistor_SMD:R_0805_2012Metric, symbol Device:R
- added R4, R5: 330, Resistor_SMD:R_0805_2012Metric, symbol Device:R
- added R6, R7: 4.7K, Resistor_SMD:R_0805_2012Metric, symbol Device:R
- added U1, U2: 24LC1025, Package_SO:SOIC-8_5.3x5.3mm_P1.27mm, symbol Memory_EEPROM:24LC1025
- added U3: ATMEGA328P-AU, Footprints:QFP80P900X900X120-32N, symbol ATMEGA328P-AU:ATMEGA328P-AU
- added U4: DS1337S_, Footprints:SOIC127P600X175-8N, symbol DS1337S_:DS1337S_
- added Y1: 32.768 KHz, Crystal:Crystal_SMD_5032-2Pin_5.0x3.2mm_HandSoldering, symbol Device:Crystal
- added Y2: 16 MHz, Crystal:Crystal_SMD_5032-2Pin_5.0x3.2mm_HandSoldering, symbol Device:Crystal
Connections:
- new net: D2.1 (K), R5.1
- new net: U4.2 (X2), Y1.1
- new net: U4.1 (X1), Y1.2
- new net: R2.2, U4.3 (~{INTA})
- new net: R3.2, U4.7 (SQW/~INT)
- new net: C2.2, U3.8 (PB7), Y2.1
- new net: C3.2, U3.7 (PB6), Y2.2
- new net: D1.1 (K), R4.2
- new net: C4.1, U3.20 (AREF)
- new net D2: U3.32 (PD2)
- new net D3: U3.1 (PD3)
- new net D4: U3.2 (PD4)
- new net D5: U3.9 (PD5)
- new net D6: U3.10 (PD6)
- new net D7: U3.11 (PD7)
- new net D8: U3.12 (PB0)
- new net GND: BT1.2 (-), C1.2, C2.1, C3.1, C4.2, C5.2, R4.1, R5.2, U1.4 (GND), U1.7 (WP), U2.2 (A1), U2.4 (GND), U2.7 (WP), U3.21 (GND), U3.3 (GND), U3.5 (GND), U4.4 (GND)
- new net MISO: U3.16 (PB4)
- new net MOSI: U3.15 (PB3)
- new net RESET: R1.2, U3.29 (PC6/~{RESET})
- new net RX: U3.30 (PD0)
- new net SCK: D1.2 (A), R6.2, U1.6 (SCL), U2.6 (SCL), U3.17 (PB5), U3.28 (PC5), U4.6 (SCL)
- new net SDA: R7.2, U1.5 (SDA), U2.5 (SDA), U3.27 (PC4), U4.5 (SDA)
- new net TX: U3.31 (PD1)
- new net VCC: BT1.1 (+), C5.1, D2.2 (A), U3.18 (AVCC), U3.4 (VCC), U3.6 (VCC)
- new net Vcc: C1.1, R1.1, R2.1, R3.1, R6.1, R7.1, U1.1 (A0), U1.2 (A1), U1.3 (A2), U1.8 (VCC), U2.1 (A0), U2.3 (A2), U2.8 (VCC), U4.8 (VCC)
- no-connect marks 0 -> 8
Other:
- added sheet connectors (connectors.kicad_sch)
- note added: "EEPROM"
- note added: "MCU"
- note added: "Mounting"
- note added: "Real time clock"
- title: (none) -> ${project_name}

Commit message: main: update schematic from 4-layer
Connections:
- net Vcc is gone; now on net VCC: C1.1, R1.1, R2.1, R3.1, R6.1, R7.1, U1.1 (A0), U1.2 (A1), U1.3 (A2), U1.8 (VCC), U2.1 (A0), U2.3 (A2), U2.8 (VCC), U4.8 (VCC)
- net SCK: no longer R6.2, U1.6 (SCL), U2.6 (SCL), U3.28 (PC5), U4.6 (SCL)
- new net SCL: R6.2, U1.6 (SCL), U2.6 (SCL), U3.28 (PC5), U4.6 (SCL)
Other:
- sheet connectors ports: added SCL; removed none
Changed lines of the file:
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@@
 		(color 0 0 0 0)
 	)
-	(junction
-		(at 255.27 40.64)
-		(diameter 0)
-		(color 0 0 0 0)
-	)
 	(no_connect
 		(at 203.2 81.28)
@@
 	(wire
 		(pts
-			(xy 134.62 143.51) (xy 140.97 143.51)
+			(xy 134.62 142.24) (xy 140.97 142.24)
 		)
 		(stroke
@@
 	(wire
 		(pts
-			(xy 134.62 140.97) (xy 140.97 140.97)
+			(xy 134.62 139.7) (xy 140.97 139.7)
 		)
 		(stroke
@@
 	(wire
 		(pts
-			(xy 259.08 40.64) (xy 255.27 40.64)
+			(xy 251.46 40.64) (xy 259.08 40.64)
 		)
 		(stroke
@@
 	(wire
 		(pts
-			(xy 184.15 66.04) (xy 184.15 67.31)
+			(xy 134.62 146.05) (xy 140.97 146.05)
 		)
 		(stroke
@@
 	(wire
 		(pts
-			(xy 113.03 46.99) (xy 119.38 46.99)
+			(xy 184.15 66.04) (xy 184.15 67.31)
 		)
 		(stroke
@@
 	(wire
 		(pts
-			(xy 203.2 93.98) (xy 203.2 99.06)
+			(xy 113.03 46.99) (xy 119.38 46.99)
 		)
 		(stroke
@@
 	(wire
 		(pts
-			(xy 233.68 48.26) (xy 233.68 50.8)
+			(xy 203.2 93.98) (xy 203.2 99.06)
 		)
 		(stroke
@@
 	(wire
 		(pts
-			(xy 233.68 99.06) (xy 238.76 99.06)
+			(xy 233.68 48.26) (xy 233.68 50.8)
 		)
 		(stroke
@@
 	(wire
 		(pts
-			(xy 196.85 55.88) (xy 185.42 55.88)
+			(xy 233.68 99.06) (xy 238.76 99.06)
 		)
 		(stroke
@@
 	(wire
 		(pts
-			(xy 170.18 147.32) (xy 176.53 147.32)
+			(xy 196.85 55.88) (xy 185.42 55.88)
 		)
 		(stroke
@@
 	(wire
 		(pts
-			(xy 195.58 76.2) (xy 184.15 76.2)
+			(xy 170.18 147.32) (xy 176.53 147.32)
 		)
 		(stroke
@@
 	(wire
 		(pts
-			(xy 255.27 40.64) (xy 251.46 40.64)
+			(xy 195.58 76.2) (xy 184.15 76.2)
 		)
 		(stroke
@@
 	)
 	(label "TX"
-		(at 134.62 140.97 180)
+		(at 134.62 139.7 180)
 		(effects
 			(font
@@
 		)
 	)
-	(label "SCK"
+	(label "SCL"
 		(at 58.42 154.94 0)
 		(effects
@@
 		)
 	)
-	(label "SCK"
+	(label "SCL"
 		(at 100.33 161.29 0)
 		(effects
@@
 		)
 	)
-	(label "SCK"
+	(label "SCL"
 		(at 134.62 134.62 180)
 		(effects
@@
 	)
 	(label "RX"
-		(at 134.62 143.51 180)
+		(at 134.62 142.24 180)
 		(effects
 			(font
@@
 		)
 	)
+	(label "SCK"
+		(at 134.62 146.05 180)
+		(effects
+			(font
+				(size 1.27 1.27)
+			)
+			(justify right bottom)
+		)
+	)
 	(label "D2"
 		(at 176.53 124.46 0)
@@
 	)
 	(label "Vcc"
+		(at 255.27 40.64 0)
+		(effects
+			(font
+				(size 1.27 1.27)
+			)
+			(justify left bottom)
+		)
+	)
+	(label "Vcc"
 		(at 81.28 139.7 0)
 		(effects
@@
 		)
 	)
-	(label "SCK"
+	(label "SCL"
 		(at 91.44 154.94 0)
 		(effects
@@
 		)
 	)
-	(label "SCK"
+	(label "SCL"
 		(at 74.93 52.07 180)
 		(effects
@@
 		)
 	)
-	(label "SCK"
+	(label "SCL"
 		(at 203.2 91.44 180)
 		(effects
@@
 	)
 	(symbol
-		(lib_id "power:PWR_FLAG")
-		(at 255.27 40.64 0)
-		(unit 1)
-		(body_style 1)
-		(exclude_from_sim no)
-		(in_bom yes)
-		(on_board yes)
-		(in_pos_files yes)
-		(dnp no)
-		(fields_autoplaced yes)
-		(property "Reference" "#FLG01"
-			(at 255.27 38.735 0)
-			(hide yes)
-			(show_name no)
-			(do_not_autoplace no)
-			(effects
-				(font
-					(size 1.27 1.27)
-				)
-			)
-		)
-		(property "Value" "PWR_FLAG"
-			(at 255.27 35.56 0)
-			(show_name no)
-			(do_not_autoplace no)
-			(effects
-				(font
-					(size 1.27 1.27)
-				)
-			)
-		)
-		(property "Footprint" ""
-			(at 255.27 40.64 0)
-			(hide yes)
-			(show_name no)
-			(do_not_autoplace no)
-			(effects
-				(font
-					(size 1.27 1.27)
-				)
-			)
-		)
-		(property "Datasheet" ""
-			(at 255.27 40.64 0)
-			(hide yes)
-			(show_name no)
-			(do_not_autoplace no)
-			(effects
-				(font
-					(size 1.27 1.27)
-				)
-			)
-		)
-		(property "Description" "Special symbol for telling ERC where power comes from"
-			(at 255.27 40.64 0)
-			(hide yes)
-			(show_name no)
-			(do_not_autoplace no)
-			(effects
-				(font
-					(size 1.27 1.27)
-				)
-			)
-		)
-		(pin "1"
-		)
-		(instances
-			(project "MCU_DataLogger"
-				(path "/eeff451f-3904-4ad2-8c5d-32d1f67f4fde"
-					(reference "#FLG01")
-					(unit 1)
-				)
-			)
-		)
-	)
-	(symbol
 		(lib_id "DS1337S_:DS1337S_")
 		(at 92.71 59.69 0)
@@
 		)
 		(pin "RX" input
-			(at 140.97 143.51 180)
+			(at 140.97 142.24 180)
 			(effects
 				(font
@@
 		)
 		(pin "SCK" passive
-			(at 140.97 134.62 180)
+			(at 140.97 146.05 180)
 			(effects
 				(font
@@
 		)
 		(pin "TX" output
-			(at 140.97 140.97 180)
+			(at 140.97 139.7 180)
 			(effects
 				(font
@@
 			(effects
 				(font
+					(size 1.27 1.27)
+				)
+				(justify left)
+			)
+		)
+		(pin "SCL" passive
+			(at 140.97 134.62 180)
+			(effects
+				(font
