File: MCU_DataLogger.kicad_pcb (KiCad board)
At the start: 2 copper layers, 0 parts

Commit message: 4-layer: start from 2-layer PCB
Parts:
- added BT1: Battery, Connector_PinHeader_2.54mm:PinHeader_1x02_P2.54mm_Vertical, F.Cu at (73.3, 87.2)
- added C1: 0.1uF, Capacitor_SMD:C_0805_2012Metric, F.Cu at (88.3, 80.9)
- added C2: 22pF, Capacitor_SMD:C_0805_2012Metric, F.Cu at (93.8, 81.0)
- added C3: 22pF, Capacitor_SMD:C_0805_2012Metric, F.Cu at (103.3, 102.6)
- added C4: 0.1uF, Capacitor_SMD:C_0805_2012Metric, F.Cu at (104.9, 98.8)
- added C5: 100nF, Capacitor_SMD:C_0805_2012Metric, F.Cu at (102.2, 81.5)
- added D1: LED, LED_SMD:LED_0805_2012Metric, F.Cu at (110.0, 81.5)
- added D2: LED, LED_SMD:LED_0805_2012Metric, F.Cu at (106.0, 81.5)
- added H1: MountingHole, MountingHole:MountingHole_2.1mm, F.Cu at (117.1, 81.5)
- added H2: MountingHole, MountingHole:MountingHole_2.1mm, F.Cu at (71.4, 81.5)
- added H3: MountingHole, MountingHole:MountingHole_2.1mm, F.Cu at (117.1, 106.9)
- added H4: MountingHole, MountingHole:MountingHole_2.1mm, F.Cu at (71.4, 106.9)
- added J1: Conn_01x04_Pin, Connector_PinHeader_2.54mm:PinHeader_1x04_P2.54mm_Vertical, F.Cu at (117.1, 94.8)
- added J2: Conn_01x04_Pin, Connector_PinHeader_2.54mm:PinHeader_1x04_P2.54mm_Vertical, F.Cu at (103.2, 106.9)
- added J3: Conn_01x09_Pin, Connector_PinHeader_2.54mm:PinHeader_1x09_P2.54mm_Vertical, F.Cu at (77.3, 106.8)
- added J4: Conn_02x03_Odd_Even, Connector_PinHeader_2.54mm:PinHeader_2x03_P2.54mm_Vertical, F.Cu at (114.6, 86.1)
- added R1: 10K, Resistor_SMD:R_0805_2012Metric, F.Cu at (110.5, 91.7)
- added R2: 10K, Resistor_SMD:R_0805_2012Metric, F.Cu at (79.4, 103.1)
- added R3: 10K, Resistor_SMD:R_0805_2012Metric, F.Cu at (83.8, 103.1)
- added R4: 330, Resistor_SMD:R_0805_2012Metric, F.Cu at (109.7, 85.3)
- added R5: 330, Resistor_SMD:R_0805_2012Metric, F.Cu at (105.7, 85.3)
- added R6: 4.7K, Resistor_SMD:R_0805_2012Metric, F.Cu at (105.1, 95.2)
- added R7: 4.7K, Resistor_SMD:R_0805_2012Metric, F.Cu at (106.7, 91.7)
- added REF**: KiCad-Logo_8mm_SilkScreen, Symbol:KiCad-Logo_8mm_SilkScreen, B.Cu at (84.8, 83.8)
- added U1: 24LC1025, Package_SO:SOIC-8_5.3x5.3mm_P1.27mm, F.Cu at (81.2, 89.8)
- added U2: 24LC1025, Package_SO:SOIC-8_5.3x5.3mm_P1.27mm, F.Cu at (81.2, 82.8)
- added U3: ATMEGA328P-AU, Footprints:QFP80P900X900X120-32N, F.Cu at (95.3, 92.2)
- added U4: DS1337S_, Footprints:SOIC127P600X175-8N, F.Cu at (81.7, 98.0)
- added Y1: 32.768 KHz, Crystal:Crystal_SMD_5032-2Pin_5.0x3.2mm_HandSoldering, F.Cu at (73.3, 98.0)
- added Y2: 16 MHz, Crystal:Crystal_SMD_5032-2Pin_5.0x3.2mm_HandSoldering, F.Cu at (94.5, 102.0)
Routing:
- net VCC: track 0.00 -> 203.3 mm, vias 0 -> 4
- net /SCL: track 0.00 -> 74.8 mm, vias 0 -> 1
- net GND: track 0.00 -> 67.8 mm, vias 0 -> 8
- net /SDA: track 0.00 -> 66.8 mm, vias 0 -> 4
- net Net-(U3-PB7): track 0.00 -> 36.5 mm, vias 0 -> 4
- net /SCK: track 0.00 -> 29.2 mm, vias 0 -> 2
- net /TX: track 0.00 -> 27.4 mm, vias 0 -> 1
- net /MOSI: track 0.00 -> 25.7 mm
- net /D3: track 0.00 -> 25.1 mm
- net /D2: track 0.00 -> 25.1 mm, vias 0 -> 1
- net /RX: track 0.00 -> 24.8 mm, vias 0 -> 1
- net /RESET: track 0.00 -> 24.2 mm, vias 0 -> 4
- net Net-(U3-PB6): track 0.00 -> 23.8 mm
- net /MISO: track 0.00 -> 22.4 mm, vias 0 -> 1
- net /D4: track 0.00 -> 22.3 mm
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- added copper zone on B.Cu, net GND
- added copper zone on F.Cu, net VCC
Other:
- board outline added: 50.8 x 30.5 mm
- board text added: "+"
- board text added: "-"
- board text added: "- 2Mbit EEPROM - RTC - I2C, SPI, GPIOs"
- board text added: "2"
- board text added: "3"
- board text added: "4"
- board text added: "5"
- board text added: "6"
- board text added: "7"
- board text added: "8"
- board text added: "Data Logger with the ATMega328P."
- board text added: "GND"
- board text added: "GPIO"
- board text added: "I2C"
- board text added: "ICSP"
- board text added: "ICSP MISO | VCC SCK | MOSI RESET | GND"
- board text added: "RX"
- board text added: "SCK"
- board text added: "SDA"
- board text added: "SERIAL"
- board text added: "TX"
- board text added: "Vcc"

Commit message: 4-layer PCB complete
Parts:
- moved C3 3.05 mm to (106.1, 101.5)
- moved C4 1.17 mm to (106.1, 98.7)
- moved R6 0.92 mm to (106.0, 95.2)
- moved R7 0.44 mm to (106.3, 91.7)
- moved R5 0.33 mm to (106.0, 85.3)
Routing:
- net VCC: track 203.3 -> 53.8 mm, vias 4 -> 8
- net GND: track 67.8 -> 46.4 mm
- net Net-(U3-PB7): track 36.5 -> 26.5 mm, vias 4 -> 3
- net /SCL: track 74.8 -> 66.1 mm, vias 1 -> 3
- net /TX: track 27.4 -> 34.9 mm, vias 1 -> 0
- net /RX: track 24.8 -> 31.3 mm, vias 1 -> 0
- net Net-(U3-PB6): track 23.8 -> 29.2 mm, vias 0 -> 3
- net /SDA: track 66.8 -> 62.1 mm, vias 4 -> 3
- net /D2: track 25.1 -> 29.3 mm, vias 1 -> 0
- net /D8: track 12.5 -> 16.1 mm, vias 1 -> 0
- net Net-(U3-AREF): track 10.3 -> 13.5 mm
- net /SCK: track 29.2 -> 32.2 mm
- net /D7: track 13.1 -> 15.1 mm, vias 1 -> 0
- net /RESET: track 24.2 -> 22.5 mm, vias 4 -> 2
- net /D6: track 13.1 -> 14.4 mm, vias 1 -> 0
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- added copper zone on In2.Cu, net VCC
- removed copper zone on F.Cu, net VCC
Other:
- board size 50.8 x 30.5 mm -> 51.7 x 31.4 mm
- copper layers 2 -> 4
