File: MCU_DataLogger.kicad_pcb (KiCad board)
At the start: 2 copper layers, 50.8 x 30.5 mm, 30 parts, among them J1 Conn_01x04_Pin, J2 Conn_01x04_Pin, J3 Conn_01x09_Pin, J4 Conn_02x03_Odd_Even, U1 24LC1025, U2 24LC1025, U3 ATMEGA328P-AU, U4 DS1337S_, Y1 32.768 KHz, Y2 16 MHz

Commit message: 2-layer PCB complete
Other:
- board size 50.8 x 30.5 mm -> 50.9 x 30.5 mm
